File: STEPBUBODC01A.kicad_sch (KiCad schematic)
At the start: 20 parts

Commit message: footprints assigned
Parts:
- removed J? (x2): Mode selection, symbol Connector:Conn_01x03_Male
- removed J? (x3): Conn_02x03_Odd_Even, symbol Connector_Generic:Conn_02x03_Odd_Even
- removed J?: Enable, symbol Connector:Conn_01x03_Male
- added J1, J3, J4: HEADER_1x03, Mlab_Pin_Headers:Straight_1x03, symbol MLAB_HEADER:HEADER_1x03
- added J2, J5, J6: HEADER_2x03_PARALLEL, Mlab_Pin_Headers:Straight_2x03, symbol MLAB_HEADER:HEADER_2x03_PARALLEL
- C1, C2, C3: renamed from C?; footprint (none) -> Mlab_C:SMD-0805
- H1, H2, H3, H4: renamed from H?; footprint (none) -> Mlab_Mechanical:MountingHole_3mm
- L1: renamed from L?; footprint (none) -> Inductor_SMD:L_1008_2520Metric
- R1, R2, R3: renamed from R?; footprint (none) -> Mlab_R:SMD-0805
- U1: renamed from U?; footprint SOTFL50P160X60-8N -> KiCad:SOTFL50P160X60-8N
- gave numbers to parts that had none: 2
Connections:
- net FB: now also J4.2
- net GND: now also J1.1, J2.1, J2.2, J2.5, J2.6, J3.1, J5.1, J5.2, J5.5, J5.6, J6.1, J6.2, J6.5, J6.6
- net V_in: now also J1.3, J3.3
- net V_out: now also J5.3, J5.4, J6.3, J6.4
- net en: now also J1.2
- net mod: now also J3.2
- net at R3.2: now also J4.1
- net at R2.2: now also J4.3
- net at F1.1: now also J2.3, J2.4
