File: STEPBUBODC01A.kicad_pcb (KiCad board)
At the start: 2 copper layers, 40.1 x 30 mm, 18 parts, among them J1 HEADER_1x03, J2 HEADER_2x03_PARALLEL, J3 HEADER_1x03, J4 HEADER_1x03, J5 HEADER_2x03_PARALLEL, J6 HEADER_2x03_PARALLEL, U1 TPS631000DRLR

Commit message: PWM/PFM label added
Other:
- board text added: "PWM/PFM"
Changed lines of the file:
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@@
     (effects (font (size 1 1) (thickness 0.15)))
   )
-  (gr_text "STEPBUBODC01A\nMLAB" (at 140.97 101.092) (layer "F.SilkS")
+  (gr_text "STEPBUBODC01A\nMLAB" (at 142.24 86.36) (layer "F.SilkS")
     (effects (font (size 1 1) (thickness 0.15)))
   )
@@
     (effects (font (size 1 1) (thickness 0.15)))
   )
+  (gr_text "PWM/PFM" (at 137.16 98.806) (layer "F.SilkS")
+    (effects (font (size 1 1) (thickness 0.15)))
+  )
