File: hw/sch_pcb/STEPBUBODC01A.kicad_pcb (KiCad board)
At the start: 2 copper layers, 40.1 x 30 mm, 18 parts, among them J1 HEADER_1x03, J2 HEADER_2x03_PARALLEL, J3 HEADER_1x03, J4 HEADER_1x03, J5 HEADER_2x03_PARALLEL, J6 HEADER_2x03_PARALLEL, U1 TPS631000DRLR

Commit message: mlab holes
Parts:
- removed H1, H2, H3, H4: MountingHole_Pad, Mlab_Mechanical:MountingHole_3mm
- added M1: HOLE M3, Mlab_Mechanical:MountingHole_3mm, F.Cu at (127.0, 76.2)
- added M2: HOLE M3, Mlab_Mechanical:MountingHole_3mm, F.Cu at (127.0, 96.5)
- added M3: HOLE, Mlab_Mechanical:MountingHole_3mm, F.Cu at (157.5, 76.2)
- added M4: HOLE, Mlab_Mechanical:MountingHole_3mm, F.Cu at (157.5, 96.5)
Changed lines of the file:
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@@
+    )
+  )
+  (footprint "Mlab_Mechanical:MountingHole_3mm" placed (layer "F.Cu")
+    (at 157.48 96.52)
+    (descr "Mounting hole, Befestigungsbohrung, 3mm, No Annular, Kein Restring,")
+    (tags "Mounting hole, Befestigungsbohrung, 3mm, No Annular, Kein Restring,")
+    (property "Sheetfile" "STEPBUBODC01A.kicad_sch")
+    (property "Sheetname" "")
+    (attr through_hole)
+    (fp_text reference "M4" (at 0 -4.191) (layer "F.SilkS") hide
+      (effects (font (size 1.524 1.524) (thickness 0.3048)))
+    )
+    (fp_text value "HOLE" (at 0 4.191) (layer "F.SilkS") hide
+      (effects (font (size 1.524 1.524) (thickness 0.3048)))
+    )
+    (fp_circle (center 0 0) (end 2.99974 0) (layer "F.Fab") (width 0.381) (fill none))
+    (pad "1" thru_hole circle (at 0 0) (size 6 6) (drill 3) (layers *.Cu *.Mask)
+      (net 2 "GND") (pintype "input") (clearance 1) (zone_connect 2))
+    (model "${MLAB}/src/3d/mechanical/m3_komplet.step"
+      (offset (xyz 0 0 0))
+      (scale (xyz 1 1 1))
+      (rotate (xyz 0 0 0))
     )
   )
@@
     )
   )
-  (footprint "Mlab_Mechanical:MountingHole_3mm" placed (layer "F.Cu")
-    (at 127 96.52)
-    (descr "Mounting hole, Befestigungsbohrung, 3mm, No Annular, Kein Restring,")
-    (tags "Mounting hole, Befestigungsbohrung, 3mm, No Annular, Kein Restring,")
-    (property "Sheetfile" "STEPBUBODC01A.kicad_sch")
-    (property "Sheetname" "")
-    (attr through_hole)
-    (fp_text reference "H3" (at 0 -4.191) (layer "F.SilkS") hide
-      (effects (font (size 1.524 1.524) (thickness 0.3048)))
-    )
-    (fp_text value "MountingHole_Pad" (at 0 4.191) (layer "F.SilkS") hide
-      (effects (font (size 1.524 1.524) (thickness 0.3048)))
-    )
-    (fp_circle (center 0 0) (end 2.99974 0) (layer "F.Fab") (width 0.381) (fill none))
-    (pad "1" thru_hole circle (at 0 0) (size 6 6) (drill 3) (layers *.Cu *.Mask)
-      (net 2 "GND") (pinfunction "1") (pintype "input") (clearance 1) (zone_connect 2))
-    (model "${MLAB}/src/3d/mechanical/m3_komplet.step"
-      (offset (xyz 0 0 0))
-      (scale (xyz 1 1 1))
-      (rotate (xyz 0 0 0))
-    )
-  )
-  (footprint "Mlab_Mechanical:MountingHole_3mm" placed (layer "F.Cu")
-    (at 157.48 76.2)
-    (descr "Mounting hole, Befestigungsbohrung, 3mm, No Annular, Kein Restring,")
-    (tags "Mounting hole, Befestigungsbohrung, 3mm, No Annular, Kein Restring,")
-    (property "Sheetfile" "STEPBUBODC01A.kicad_sch")
-    (property "Sheetname" "")
-    (attr through_hole)
-    (fp_text reference "H4" (at 0 -4.191) (layer "F.SilkS") hide
-      (effects (font (size 1.524 1.524) (thickness 0.3048)))
-    )
-    (fp_text value "MountingHole_Pad" (at 0 4.191) (layer "F.SilkS") hide
-      (effects (font (size 1.524 1.524) (thickness 0.3048)))
-    )
-    (fp_circle (center 0 0) (end 2.99974 0) (layer "F.Fab") (width 0.381) (fill none))
-    (pad "1" thru_hole circle (at 0 0) (size 6 6) (drill 3) (layers *.Cu *.Mask)
-      (net 2 "GND") (pinfunction "1") (pintype "input") (clearance 1) (zone_connect 2))
-    (model "${MLAB}/src/3d/mechanical/m3_komplet.step"
-      (offset (xyz 0 0 0))
-      (scale (xyz 1 1 1))
-      (rotate (xyz 0 0 0))
-    )
-  )
   (footprint "Mlab_Pin_Headers:Straight_1x03" (layer "F.Cu")
     (at 137.16 76.2 -90)
@@
   )
   (footprint "Mlab_Mechanical:MountingHole_3mm" placed (layer "F.Cu")
-    (at 157.48 96.52)
-    (descr "Mounting hole, Befestigungsbohrung, 3mm, No Annular, Kein Restring,")
-    (tags "Mounting hole, Befestigungsbohrung, 3mm, No Annular, Kein Restring,")
-    (property "Sheetfile" "STEPBUBODC01A.kicad_sch")
-    (property "Sheetname" "")
-    (attr through_hole)
-    (fp_text reference "H2" (at 0 -4.191) (layer "F.SilkS") hide
-      (effects (font (size 1.524 1.524) (thickness 0.3048)))
-    )
-    (fp_text value "MountingHole_Pad" (at 0 4.191) (layer "F.SilkS") hide
-      (effects (font (size 1.524 1.524) (thickness 0.3048)))
-    )
-    (fp_circle (center 0 0) (end 2.99974 0) (layer "F.Fab") (width 0.381) (fill none))
-    (pad "1" thru_hole circle (at 0 0) (size 6 6) (drill 3) (layers *.Cu *.Mask)
-      (net 2 "GND") (pinfunction "1") (pintype "input") (clearance 1) (zone_connect 2))
+    (at 127 76.2)
+    (descr "Mounting hole, Befestigungsbohrung, 3mm, No Annular, Kein Restring,")
+    (tags "Mounting hole, Befestigungsbohrung, 3mm, No Annular, Kein Restring,")
+    (property "Sheetfile" "STEPBUBODC01A.kicad_sch")
+    (property "Sheetname" "")
+    (attr through_hole)
+    (fp_text reference "M1" (at 0 -4.191) (layer "F.SilkS") hide
+      (effects (font (size 1.524 1.524) (thickness 0.3048)))
+    )
+    (fp_text value "HOLE M3" (at 0 4.191) (layer "F.SilkS") hide
+      (effects (font (size 1.524 1.524) (thickness 0.3048)))
+    )
+    (fp_circle (center 0 0) (end 2.99974 0) (layer "F.Fab") (width 0.381) (fill none))
+    (pad "1" thru_hole circle (at 0 0) (size 6 6) (drill 3) (layers *.Cu *.Mask)
+      (net 2 "GND") (pintype "input") (clearance 1) (zone_connect 2))
+    (model "${MLAB}/src/3d/mechanical/m3_komplet.step"
+      (offset (xyz 0 0 0))
+      (scale (xyz 1 1 1))
+      (rotate (xyz 0 0 0))
+    )
+  )
+  (footprint "Mlab_Mechanical:MountingHole_3mm" placed (layer "F.Cu")
+    (at 127 96.52)
+    (descr "Mounting hole, Befestigungsbohrung, 3mm, No Annular, Kein Restring,")
+    (tags "Mounting hole, Befestigungsbohrung, 3mm, No Annular, Kein Restring,")
+    (property "Sheetfile" "STEPBUBODC01A.kicad_sch")
+    (property "Sheetname" "")
+    (attr through_hole)
+    (fp_text reference "M2" (at 0 -4.191) (layer "F.SilkS") hide
+      (effects (font (size 1.524 1.524) (thickness 0.3048)))
+    )
+    (fp_text value "HOLE M3" (at 0 4.191) (layer "F.SilkS") hide
+      (effects (font (size 1.524 1.524) (thickness 0.3048)))
+    )
+    (fp_circle (center 0 0) (end 2.99974 0) (layer "F.Fab") (width 0.381) (fill none))
+    (pad "1" thru_hole circle (at 0 0) (size 6 6) (drill 3) (layers *.Cu *.Mask)
+      (net 2 "GND") (pintype "input") (clearance 1) (zone_connect 2))
     (model "${MLAB}/src/3d/mechanical/m3_komplet.step"
       (offset (xyz 0 0 0))
@@
   )
   (footprint "Mlab_Mechanical:MountingHole_3mm" placed (layer "F.Cu")
-    (at 127 76.2)
-    (descr "Mounting hole, Befestigungsbohrung, 3mm, No Annular, Kein Restring,")
-    (tags "Mounting hole, Befestigungsbohrung, 3mm, No Annular, Kein Restring,")
-    (property "Sheetfile" "STEPBUBODC01A.kicad_sch")
-    (property "Sheetname" "")
-    (attr through_hole)
-    (fp_text reference "H1" (at 0 -4.191) (layer "F.SilkS") hide
-      (effects (font (size 1.524 1.524) (thickness 0.3048)))
-    )
-    (fp_text value "MountingHole_Pad" (at 0 4.191) (layer "F.SilkS") hide
-      (effects (font (size 1.524 1.524) (thickness 0.3048)))
-    )
-    (fp_circle (center 0 0) (end 2.99974 0) (layer "F.Fab") (width 0.381) (fill none))
-    (pad "1" thru_hole circle (at 0 0) (size 6 6) (drill 3) (layers *.Cu *.Mask)
-      (net 2 "GND") (pinfunction "1") (pintype "input") (clearance 1) (zone_connect 2))
-    (model "${MLAB}/src/3d/mechanical/m3_komplet.step"
-      (offset (xyz 0 0 0))
+    (at 157.48 76.2)
+    (descr "Mounting hole, Befestigungsbohrung, 3mm, No Annular, Kein Restring,")
+    (tags "Mounting hole, Befestigungsbohrung, 3mm, No Annular, Kein Restring,")
+    (property "Sheetfile" "STEPBUBODC01A.kicad_sch")
+    (property "Sheetname" "")
+    (attr through_hole)
+    (fp_text reference "M3" (at 0 -4.191) (layer "F.SilkS") hide
+      (effects (font (size 1.524 1.524) (thickness 0.3048)))
+    )
+    (fp_text value "HOLE" (at 0 4.191) (layer "F.SilkS") hide
+      (effects (font (size 1.524 1.524) (thickness 0.3048)))
+    )
+    (fp_circle (center 0 0) (end 2.99974 0) (layer "F.Fab") (width 0.381) (fill none))
+    (pad "1" thru_hole circle (at 0 0) (size 6 6) (drill 3) (layers *.Cu *.Mask)
+      (net 2 "GND") (pintype "input") (clearance 1) (zone_connect 2))
+    (model "${MLAB}/src/3d/mechanical/m3_komplet.step"
+      (offset (xyz 0 0 0))
