File: hw/sch_pcb/STEPBUBODC01A.kicad_sch (KiCad schematic)
At the start: 20 parts, among them J1 HEADER_1x03, J2 HEADER_2x03_PARALLEL, J3 HEADER_1x03, J4 HEADER_1x03, J5 HEADER_2x03_PARALLEL, J6 HEADER_2x03_PARALLEL, U1 TPS631000DRLR

Commit message: mlab holes
Parts:
- removed H1, H2, H3, H4: MountingHole_Pad, Mlab_Mechanical:MountingHole_3mm, symbol Mechanical:MountingHole_Pad
- added M1, M2: HOLE M3, Mlab_Mechanical:MountingHole_3mm, symbol mlab-default-rescue:HOLE
- added M3, M4: HOLE, Mlab_Mechanical:MountingHole_3mm, symbol mlab-default-rescue:HOLE
Connections:
- net GND: now also M1.1, M2.1, M3.1, M4.1
Other:
- note added: "MOUNTING HOLES"
- note removed: "Mounting holes"
